File: USB_CHARGER_LITHIUM/USB_CHARGER_LITHIUM.kicad_pcb (KiCad board)
At the start: 2 copper layers, 57.2 x 30.5 mm, 21 parts, among them J1 USB4135, J2 Conn_01x02, J3 Conn_01x02, U1 TP5000X-4.2-ESOP8, U2 XB7608A

Commit message: Rev 1.1
Parts:
- H1, H2: footprint MountingHole:MountingHole_3.2mm_M3_DIN965_Pad -> MountingHole:MountingHole_4.3mm_M4_Pad_Via
- renumbered D3 to SS34, U1 to TP5000, U2 to XB7608A
Routing:
- net GND: track 0.01 -> 0.17 mm, vias 143 -> 104
- net GNDPWR: vias 12 -> 9
- net (no net): vias 5 -> 0
Other:
- board text added: "REV 1.1"
- board text removed: "REV 1.0"
